Commit message: [ADD] added the environment

File: fmauch_universal_robot/ur_description/urdf/ur5e.xacro (robot description, xacro)
@@ -4,4 +4,5 @@
 <xacro:include filename="$(find ur_description)/urdf/inc/ur5e_macro.xacro"/>
 <xacro:include filename="$(find robotiq_2f_85_gripper_visualization)/urdf/robotiq_arg2f_85_model_macro.xacro" />
+<xacro:include filename="$(find ur_description)/urdf/environment.xacro"/>
 <!-- create the robot + eef combo itself as a macro -->
 <xacro:macro name="ee_robot" params="prefix">
@@ -9,4 +10,5 @@
   <xacro:ur5e_robot prefix="${prefix}robot_"/>
   <xacro:robotiq_arg2f_85 prefix="${prefix}gripper_" />
+  <xacro:environment prefix="${prefix}env_"/>
   <!-- attach gripper -->
   <joint name="${prefix}robot_tool0-${prefix}gripper_robotiq_arg2f_base_link" type="fixed">
@@ -15,4 +17,10 @@
     <child link="${prefix}gripper_robotiq_arg2f_base_link" />
   </joint>
+  <!-- env -->
+  <joint name="${prefix}env_to_robot" type="fixed">
+    <origin xyz="0 0 0" rpy="0 0 0" />
+    <parent link="${prefix}env_table_base"/>
+    <child link="${prefix}robot_base_link" />
+  </joint>
 </xacro:macro>
 <xacro:ee_robot prefix=""/>
