Commit message: [ADD] fix & updates of env and gripper

File: fmauch_universal_robot/ur_description/urdf/ur5e_mlp3240_env.xacro (robot description, xacro)
@@ -19,5 +19,5 @@
   <!-- env -->
   <joint name="${prefix}env_to_robot" type="fixed">
-    <origin xyz="0.0425 -0.0925  0" rpy="0 0 0"/>
+    <origin xyz="0.0425 -0.0925  0.015" rpy="0 0 0"/>
     <parent link="${prefix}env_table_base"/>
     <child link="${prefix}robot_base_link" />

File: mlp3240_visual/urdf/mlp3240_macro.xacro (robot description, xacro)
@@ -53,5 +53,5 @@
                     <origin xyz="0 0.005 0.0065" rpy="0 0 1.57" />
                     <geometry>
-                        <mesh filename="package://mlp3240_visual/mesh/visual/front.stl" scale="0.001 0.001 0.001"/>
+                        <mesh filename="package://mlp3240_visual/mesh/visual/front_w_box.stl" scale="0.001 0.001 0.001"/>
                     </geometry>
                     <material name="black">
@@ -75,5 +75,5 @@
                     <origin xyz="0.015 0 0.001" rpy="0 0 1.57" />
                     <geometry>
-                        <mesh filename="package://mlp3240_visual/mesh/visual/finger.stl" scale="0.001 0.001 0.001"/>
+                        <mesh filename="package://mlp3240_visual/mesh/visual/finger_1.stl" scale="0.001 0.001 0.001"/>
                     </geometry>
                     <material name="white"/>
@@ -84,5 +84,5 @@
                     <origin xyz="0.015 0 0.001" rpy="0 0 1.57" />
                     <geometry>
-                        <mesh filename="package://mlp3240_visual/mesh/visual/finger.stl" scale="0.001 0.001 0.001"/>
+                        <mesh filename="package://mlp3240_visual/mesh/visual/finger_2.stl" scale="0.001 0.001 0.001"/>
                     </geometry>
                     <material name="white"/>
