Commit message: [FIX] fixed some stuff of tf

File: fmauch_universal_robot/ur_description/urdf/environment.xacro (robot description, xacro)
@@ -9,4 +9,7 @@
       </geometry>
       <origin xyz="0 0 -0.05" rpy='0 0 0'/>
+      <material name="orange">
+          <color rgba="${255/255} ${84/255} ${1/255} 1.0"/>
+      </material>
     </visual>
   </link>
@@ -16,5 +19,8 @@
         <box size='1.0 5.0 0.05'/>
       </geometry>
-      <origin xyz="-1.05 0 -0.05" rpy='0 0 0'/>
+      <material name="green">
+          <color rgba="${8/255} ${238/255} ${1/255} 1.0"/>
+      </material>
+      <origin xyz="0 0 0" rpy='0 0 0'/>
     </visual>
   </link>
@@ -24,5 +30,8 @@
         <box size='1.5 0.75 0.05'/>
       </geometry>
-      <origin xyz="0.25 -0.9 -0.05" rpy='0 0 0'/>
+      <material name="green">
+          <color rgba="${8/255} ${238/255} ${1/255} 1.0"/>
+      </material>
+      <origin xyz="0 0 0" rpy='0 0 0'/>
     </visual>
   </link>
@@ -32,5 +41,8 @@
         <box size='4 0.05 1.5'/>
       </geometry>
-      <origin xyz="0.25 0.75 -0.05" rpy='0 0 0'/>
+      <origin xyz="0 0 0" rpy='0 0 0'/>
+      <material name="yellow">
+          <color rgba="${222/255} ${247/255} ${1/255} 1.0"/>
+      </material>
     </visual>
   </link>
@@ -40,32 +52,30 @@
         <box size='0.05 1.2 1.5'/>
       </geometry>
-      <origin xyz="0.55 0.12 -0.05" rpy='0 0 0'/>
+      <origin xyz="0 0 0" rpy='0 0 0'/>
+      <material name="yellow">
+          <color rgba="${222/255} ${247/255} ${1/255} 1.0"/>
+      </material>
     </visual>
   </link>
-  <joint name="${prefix}table_base" type="fixed">
+  <joint name="${prefix}conveyor_base_joint" type="fixed">
     <parent link="${prefix}table_base"/>
     <child link="${prefix}conveyor_base"/>
-    <origin xyz="0 0 0" rpy='0 0 0'/>
+    <origin xyz="-1.05 0 -0.05" rpy='0 0 0'/>
   </joint>
-  <joint name="${prefix}conveyor_base" type="fixed">
+  <joint name="${prefix}conveyor_to_visual_inspection_joint" type="fixed">
     <parent link="${prefix}table_base"/>
     <child link="${prefix}conveyor_to_visual_inspection"/>
-    <origin xyz="0 0 0" rpy='0 0 0'/>
+     <origin xyz="0.25 -0.9 -0.05"  rpy='0 0 0'/>
   </joint>
-  <joint name="${prefix}conveyor_to_visual_inspection" type="fixed">
+  <joint name="${prefix}wall_1_joint" type="fixed">
     <parent link="${prefix}table_base"/>
     <child link="${prefix}wall_1"/>
-     <origin xyz="0 0 0"  rpy='0 0 0'/>
+    <origin xyz="0.25 0.75 -0.05"  rpy='0 0 0'/>
   </joint>
-  <joint name="${prefix}wall_1" type="fixed">
+  <joint name="${prefix}wall_2_joint" type="fixed">
     <parent link="${prefix}table_base"/>
     <child link="${prefix}wall_2"/>
-    <origin xyz="0 0 0"  rpy='0 0 0'/>
-  </joint>
-  <joint name="${prefix}wall_2" type="fixed">
-    <parent link="${prefix}table_base"/>
-    <child link="${prefix}wall_2"/>
-    <origin xyz="0 0 0"  rpy='0 0 0'/>
+    <origin xyz="0.55 0.12 -0.05"  rpy='0 0 0'/>
   </joint>
 </xacro:macro>
-  </robot>
+</robot>

Commit message: [ADD] better modellation of ice-lab environment

File: fmauch_universal_robot/ur_description/urdf/environment.xacro (robot description, xacro)
@@ -1,14 +1,23 @@
 <robot xmlns:xacro="http://wiki.ros.org/xacro">>
-<xacro:macro name="environment" params="
-    prefix "
-  >
-<link name="${prefix}table_base">
+<xacro:macro name="environment" params="prefix">
+  <link name="${prefix}table_base">
     <visual>
       <geometry>
-        <box size='1.0 1.0 0.05'/>
+        <mesh filename="package://ur_description/meshes/ur5e/visual/table.stl" scale="0.01 0.01 0.021"/>
       </geometry>
-      <origin xyz="0 0 -0.05" rpy='0 0 0'/>
+      <origin xyz="0 0 0" rpy='0 0 0'/>
       <material name="orange">
           <color rgba="${255/255} ${84/255} ${1/255} 1.0"/>
+      </material>
+    </visual>
+  </link>
+  <link name="${prefix}floor">
+    <visual>
+      <geometry>
+        <mesh filename="package://ur_description/meshes/ur5e/visual/floor.stl" scale="0.1 0.1 0.1"/>
+      </geometry>
+      <origin xyz="0 0 0" rpy='0 0 0'/>
+      <material name="gray">
+          <color rgba="${156/255} ${134/255} ${92/255} 1.0"/>
       </material>
     </visual>
@@ -17,5 +26,5 @@
     <visual>
       <geometry>
-        <box size='1.0 5.0 0.05'/>
+          <mesh filename="package://ur_description/meshes/ur5e/visual/conveyor_test.stl" scale="0.03 0.01 0.01"/>
       </geometry>
       <material name="green">
@@ -27,7 +36,7 @@
   <link name="${prefix}conveyor_to_visual_inspection">
     <visual>
-      <geometry>
-        <box size='1.5 0.75 0.05'/>
-      </geometry>
+        <geometry>
+          <mesh filename="package://ur_description/meshes/ur5e/visual/conveyor_test.stl" scale="0.01 0.01 0.01"/>
+        </geometry>
       <material name="green">
           <color rgba="${8/255} ${238/255} ${1/255} 1.0"/>
@@ -58,13 +67,18 @@
     </visual>
   </link>
+  <joint name="${prefix}floor_joint" type="fixed">
+    <parent link="${prefix}table_base"/>
+    <child link="${prefix}floor"/>
+    <origin xyz="0 0 -0.81" rpy='0 0 0'/>
+  </joint>
   <joint name="${prefix}conveyor_base_joint" type="fixed">
     <parent link="${prefix}table_base"/>
     <child link="${prefix}conveyor_base"/>
-    <origin xyz="-1.05 0 -0.05" rpy='0 0 0'/>
+    <origin xyz="-1.05 0 -0.75" rpy='0 0 -1.57'/>
   </joint>
   <joint name="${prefix}conveyor_to_visual_inspection_joint" type="fixed">
     <parent link="${prefix}table_base"/>
     <child link="${prefix}conveyor_to_visual_inspection"/>
-     <origin xyz="0.25 -0.9 -0.05"  rpy='0 0 0'/>
+     <origin xyz="0.25 -0.9 -0.75"  rpy='0 0 0'/>
   </joint>
   <joint name="${prefix}wall_1_joint" type="fixed">

Commit message: [ADD] added the model of the mlp3240

File: fmauch_universal_robot/ur_description/urdf/environment.xacro (robot description, xacro)
@@ -1,3 +1,3 @@
-<robot xmlns:xacro="http://wiki.ros.org/xacro">>
+<robot xmlns:xacro="http://wiki.ros.org/xacro">
 <xacro:macro name="environment" params="prefix">
   <link name="${prefix}table_base">
@@ -82,13 +82,15 @@
      <origin xyz="0.25 -0.9 -0.75"  rpy='0 0 0'/>
   </joint>
-  <joint name="${prefix}wall_1_joint" type="fixed">
+  <joint name="${prefix}wall_1_joint" type="prismatic">
     <parent link="${prefix}table_base"/>
     <child link="${prefix}wall_1"/>
     <origin xyz="0.25 0.75 -0.05"  rpy='0 0 0'/>
+    <limit effort="1000.0" lower="-0.38" upper="0" velocity="0.5"/>
   </joint>
-  <joint name="${prefix}wall_2_joint" type="fixed">
+  <joint name="${prefix}wall_2_joint" type="prismatic">
     <parent link="${prefix}table_base"/>
     <child link="${prefix}wall_2"/>
     <origin xyz="0.55 0.12 -0.05"  rpy='0 0 0'/>
+    <limit effort="1000.0" lower="-0.38" upper="0" velocity="0.5"/>
   </joint>
 </xacro:macro>

Commit message: [FIX] fixed the trajectory of pick and place

File: fmauch_universal_robot/ur_description/urdf/environment.xacro (robot description, xacro)
@@ -4,5 +4,6 @@
     <visual>
       <geometry>
-        <mesh filename="package://ur_description/meshes/ur5e/visual/table.stl" scale="0.01 0.01 0.021"/>
+        <!-- <mesh filename="package://ur_description/meshes/ur5e/visual/table.stl" scale="0.01 0.01 0.021"/> -->
+        <box size="0.66 0.66 0.05"/>
       </geometry>
       <origin xyz="0 0 0" rpy='0 0 0'/>
@@ -26,5 +27,6 @@
     <visual>
       <geometry>
-          <mesh filename="package://ur_description/meshes/ur5e/visual/conveyor_test.stl" scale="0.03 0.01 0.01"/>
+        <box size="2 0.25 0.05"/>
+        <!-- <mesh filename="package://ur_description/meshes/ur5e/visual/conveyor_test.stl" scale="0.03 0.01 0.01"/> -->
       </geometry>
       <material name="green">
@@ -37,5 +39,6 @@
     <visual>
         <geometry>
-          <mesh filename="package://ur_description/meshes/ur5e/visual/conveyor_test.stl" scale="0.01 0.01 0.01"/>
+          <box size="1 0.25 0.05"/>
+          <!-- <mesh filename="package://ur_description/meshes/ur5e/visual/conveyor_test.stl" scale="0.01 0.01 0.01"/> -->
         </geometry>
       <material name="green">
@@ -59,5 +62,5 @@
     <visual>
       <geometry>
-        <box size='0.05 1.2 1.5'/>
+        <box size='0.05 0.85 1.5'/>
       </geometry>
       <origin xyz="0 0 0" rpy='0 0 0'/>
@@ -70,27 +73,25 @@
     <parent link="${prefix}table_base"/>
     <child link="${prefix}floor"/>
-    <origin xyz="0 0 -0.81" rpy='0 0 0'/>
+    <origin xyz="0 0 -0.75" rpy='0 0 0'/>
   </joint>
   <joint name="${prefix}conveyor_base_joint" type="fixed">
     <parent link="${prefix}table_base"/>
     <child link="${prefix}conveyor_base"/>
-    <origin xyz="-1.05 0 -0.75" rpy='0 0 -1.57'/>
+    <origin xyz="-0.45 0 0" rpy='0 0 -1.57'/>
   </joint>
   <joint name="${prefix}conveyor_to_visual_inspection_joint" type="fixed">
     <parent link="${prefix}table_base"/>
     <child link="${prefix}conveyor_to_visual_inspection"/>
-     <origin xyz="0.25 -0.9 -0.75"  rpy='0 0 0'/>
+     <origin xyz="0.25 -0.45 0"  rpy='0 0 0'/>
   </joint>
-  <joint name="${prefix}wall_1_joint" type="prismatic">
+  <joint name="${prefix}wall_1_joint" type="fixed">
     <parent link="${prefix}table_base"/>
     <child link="${prefix}wall_1"/>
-    <origin xyz="0.25 0.75 -0.05"  rpy='0 0 0'/>
-    <limit effort="1000.0" lower="-0.38" upper="0" velocity="0.5"/>
+    <origin xyz="0.25 0.6 0"  rpy='0 0 0'/>
   </joint>
-  <joint name="${prefix}wall_2_joint" type="prismatic">
+  <joint name="${prefix}wall_2_joint" type="fixed">
     <parent link="${prefix}table_base"/>
     <child link="${prefix}wall_2"/>
-    <origin xyz="0.55 0.12 -0.05"  rpy='0 0 0'/>
-    <limit effort="1000.0" lower="-0.38" upper="0" velocity="0.5"/>
+    <origin xyz="0.4 0.12 0"  rpy='0 0 0'/>
   </joint>
 </xacro:macro>

File: fmauch_universal_robot/ur_description/urdf/ur5e.xacro (robot description, xacro)
@@ -19,7 +19,7 @@
   <!-- env -->
   <joint name="${prefix}env_to_robot" type="fixed">
-    <origin xyz="0 0 0" rpy="0 0 0" />
+    <origin xyz="0.25 -1.5 0" rpy="0 0 0"/>
     <parent link="${prefix}env_table_base"/>
-    <child link="${prefix}robot_base_link" />
+    <child link="${prefix}robot_base_link"/>
   </joint>
 </xacro:macro>

File: fmauch_universal_robot/ur_description/urdf/ur5e_mlp3240_env.xacro (robot description, xacro)
@@ -19,5 +19,5 @@
   <!-- env -->
   <joint name="${prefix}env_to_robot" type="fixed">
-    <origin xyz="0 0 0" rpy="0 0 0" />
+    <origin xyz="0.0425 -0.0925  0" rpy="0 0 0"/>
     <parent link="${prefix}env_table_base"/>
     <child link="${prefix}robot_base_link" />

Commit message: [UP] updated all the tasks and meshes

File: fmauch_universal_robot/ur_description/urdf/environment.xacro (robot description, xacro)
@@ -4,5 +4,5 @@
     <visual>
       <geometry>
-        <!-- <mesh filename="package://ur_description/meshes/ur5e/visual/table.stl" scale="0.01 0.01 0.021"/> -->
+        <mesh filename="package://ur_description/meshes/ur5e/visual/table.stl"/>
         <box size="0.66 0.66 0.05"/>
       </geometry>
@@ -27,6 +27,6 @@
     <visual>
       <geometry>
-        <box size="2 0.25 0.05"/>
-        <!-- <mesh filename="package://ur_description/meshes/ur5e/visual/conveyor_test.stl" scale="0.03 0.01 0.01"/> -->
+        <!-- <box size="2 0.25 0.05"/> -->
+        <mesh filename="package://ur_description/meshes/ur5e/visual/conveyor_ice.stl" />
       </geometry>
       <material name="green">
@@ -39,6 +39,6 @@
     <visual>
         <geometry>
-          <box size="1 0.25 0.05"/>
-          <!-- <mesh filename="package://ur_description/meshes/ur5e/visual/conveyor_test.stl" scale="0.01 0.01 0.01"/> -->
+          <!-- <box size="1 0.25 0.05"/> -->
+          <mesh filename="package://ur_description/meshes/ur5e/visual/conveyor_iceLab_visual.stl"/>
         </geometry>
       <material name="green">
@@ -70,4 +70,26 @@
     </visual>
   </link>
+  <link name="${prefix}pick_slab_visual">
+    <visual>
+      <geometry>
+        <box size="0.25 0.25 0.03"/>
+      </geometry>
+      <origin xyz="0 0 0" rpy='0 0 0'/>
+      <material name="orange">
+          <color rgba="${255/255} ${84/255} ${1/255} 1.0"/>
+      </material>
+    </visual>
+  </link>
+  <link name="${prefix}pick_slab">
+    <visual>
+      <geometry>
+        <box size="0.25 0.25 0.03"/>
+      </geometry>
+      <origin xyz="0 0 0" rpy='0 0 0'/>
+      <material name="orange">
+          <color rgba="${255/255} ${84/255} ${1/255} 1.0"/>
+      </material>
+    </visual>
+  </link>
   <joint name="${prefix}floor_joint" type="fixed">
     <parent link="${prefix}table_base"/>
@@ -85,4 +107,14 @@
      <origin xyz="0.25 -0.45 0"  rpy='0 0 0'/>
   </joint>
+  <joint name="${prefix}visual_slab_joint" type="fixed">
+    <parent link="${prefix}conveyor_to_visual_inspection"/>
+    <child link="${prefix}pick_slab_visual"/>
+     <origin xyz="0 0 0.01"  rpy='0 0 0'/>
+  </joint>
+  <joint name="${prefix}pick_slab_joint" type="fixed">
+    <parent link="${prefix}conveyor_base"/>
+    <child link="${prefix}pick_slab"/>
+     <origin xyz="0.1 0 0.01"  rpy='0 0 0'/>
+  </joint>
   <joint name="${prefix}wall_1_joint" type="fixed">
     <parent link="${prefix}table_base"/>

File: fmauch_universal_robot/ur_description/urdf/ur5e_mlp3240_env.xacro (robot description, xacro)
@@ -19,5 +19,5 @@
   <!-- env -->
   <joint name="${prefix}env_to_robot" type="fixed">
-    <origin xyz="0.0425 -0.0925  0.015" rpy="0 0 0"/>
+    <origin xyz="0.0425 -0.0925  0" rpy="0 0 0"/>
     <parent link="${prefix}env_table_base"/>
     <child link="${prefix}robot_base_link" />

Commit message: [UP] updated pick_place & glue sealing

File: fmauch_universal_robot/ur_description/urdf/environment.xacro (robot description, xacro)
@@ -51,5 +51,5 @@
     <visual>
       <geometry>
-        <box size='4 0.05 1.5'/>
+        <box size='4 0.05 4.5'/>
       </geometry>
       <origin xyz="0 0 0" rpy='0 0 0'/>
@@ -62,5 +62,5 @@
     <visual>
       <geometry>
-        <box size='0.05 0.85 1.5'/>
+        <box size='0.05 0.85 4.5'/>
       </geometry>
       <origin xyz="0 0 0" rpy='0 0 0'/>
@@ -120,10 +120,10 @@
     <parent link="${prefix}table_base"/>
     <child link="${prefix}wall_1"/>
-    <origin xyz="0.25 0.6 0"  rpy='0 0 0'/>
+    <origin xyz="0.25 0.3 0"  rpy='0 0 0'/>
   </joint>
   <joint name="${prefix}wall_2_joint" type="fixed">
     <parent link="${prefix}table_base"/>
     <child link="${prefix}wall_2"/>
-    <origin xyz="0.4 0.12 0"  rpy='0 0 0'/>
+    <origin xyz="0.25 0.25 0"  rpy='0 0 0'/>
   </joint>
 </xacro:macro>

Commit message: [UP] updated and corrected minor stuff

File: fmauch_universal_robot/ur_description/urdf/environment.xacro (robot description, xacro)
@@ -125,5 +125,5 @@
     <parent link="${prefix}table_base"/>
     <child link="${prefix}wall_2"/>
-    <origin xyz="0.25 0.25 0"  rpy='0 0 0'/>
+    <origin xyz="0.25 0.35 0"  rpy='0 0 0'/>
   </joint>
 </xacro:macro>

Commit message: [FIX] environment fix

File: fmauch_universal_robot/ur_description/urdf/environment.xacro (robot description, xacro)
@@ -100,10 +100,10 @@
     <parent link="${prefix}table_base"/>
     <child link="${prefix}conveyor_base"/>
-    <origin xyz="-0.45 0 0" rpy='0 0 -1.57'/>
+    <origin xyz="-0.45 0 0.05" rpy='0 0 -1.57'/>
   </joint>
   <joint name="${prefix}conveyor_to_visual_inspection_joint" type="fixed">
     <parent link="${prefix}table_base"/>
     <child link="${prefix}conveyor_to_visual_inspection"/>
-     <origin xyz="0.25 -0.45 0"  rpy='0 0 0'/>
+     <origin xyz="0.25 -0.45 0.05"  rpy='0 0 0'/>
   </joint>
   <joint name="${prefix}visual_slab_joint" type="fixed">
