Commit message: [ADD] added the image folder for readme

File: mlp3240_visual/urdf/mlp3240_macro.xacro (robot description, xacro)
@@ -105,5 +105,5 @@
             <parent link="top"/>
             <child link="finger1"/>
-            <origin xyz="${physical_parameters['top_x']/2 - 0.005} 0 0.021" rpy='0 0 -3.14'/>
+            <origin xyz="${physical_parameters['top_x']/2 - 0.005} 0 0.0211" rpy='0 0 -3.14'/>
             <limit upper="0.042" lower="0.0" effort="300" velocity="1"/>
         </joint>
