Commit message: [ADD] added mesh & other stuff related to mlp3240

File: mlp3240_visual/urdf/mlp3240.xacro (robot description, xacro)
@@ -1,13 +1,13 @@
 <robot name="mpl3240" xmlns:xacro="http://ros.org/wiki/xacro">
     <xacro:include filename="$(find mlp3240_visual)/urdf/mlp3240_macro.xacro"/>
-    <xacro:macro name="mlp_3240_world">
-        <xacro:mlp3240/>
+    <xacro:macro name="mlp_3240_world" params="prefix">
+        <xacro:mlp3240 prefix="${prefix}"/>
         <link name="map"/>
-        <joint name="base_to_world_joint" type="fixed">
+        <joint name="${prefix}base_to_world_joint" type="fixed">
             <parent link="map"/>
-            <child link="base_link"/>
+            <child link="${prefix}base_link"/>
             <origin xyz="0 0 0" rpy="0 0 0"/>
         </joint>
     </xacro:macro>
-    <xacro:mlp_3240_world/>
+    <xacro:mlp_3240_world prefix="gripper_"/>
 </robot>
